Commit message: exp_climbench

File: Agent/Component_asset/2wheels_urdf/wheel_only.urdf (robot description, URDF)
Before this commit: robot wheel_only, 2 links, 1 joints
Links:
- link wheel: geometry collision mesh filename=package://assets/wheel.stl scale=4 4 4; visual mesh filename=package://assets/wheel.stl scale=4 4 4
Joints:
- joint wheel_to_cylinder: origin xyz=0 0 0.015 rpy=0 0 0 -> xyz=0 0 0.012 rpy=0 0 0
